File: power_distribution/hw/power_distribution/stage1.kicad_sch (KiCad schematic)
At the start: 1 part

Commit message: Finish output stage
Parts:
- removed U?: LMR51635XFDDCR, DDC0006A-MFG, symbol LMR51635XFDDCR:LMR51635XFDDCR
- added U1: LMR51635XFDDCR, DDC0006A-MFG, symbol LMR51635XFDDCR:LMR51635XFDDCR
Changed lines of the file:
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@@
 	(hierarchical_label "VOUT"
 		(shape output)
-		(at 220.98 93.98 0)
+		(at 95.25 50.8 0)
 		(effects
 			(font
@@
 	(hierarchical_label "VIN"
 		(shape input)
-		(at 52.07 83.82 180)
+		(at 38.1 44.45 180)
 		(effects
 			(font
@@
 	(symbol
 		(lib_id "LMR51635XFDDCR:LMR51635XFDDCR")
-		(at 58.42 41.91 0)
+		(at 48.26 44.45 0)
 		(unit 1)
 		(exclude_from_sim no)
@@
 		(dnp no)
 		(fields_autoplaced yes)
-		(property "Reference" "U?"
-			(at 73.66 31.75 0)
+		(property "Reference" "U1"
+			(at 63.5 34.29 0)
 			(effects
 				(font
@@
 		)
 		(property "Value" "LMR51635XFDDCR"
-			(at 73.66 34.29 0)
+			(at 63.5 36.83 0)
 			(effects
 				(font
@@
 		)
 		(property "Footprint" "DDC0006A-MFG"
-			(at 58.42 41.91 0)
+			(at 48.26 44.45 0)
 			(effects
 				(font
@@
 		)
 		(property "Datasheet" "https://www.ti.com/lit/gpn/lmr51635"
-			(at 58.42 41.91 0)
+			(at 48.26 44.45 0)
 			(effects
 				(font
@@
 		)
 		(property "Description" ""
-			(at 58.42 41.91 0)
+			(at 48.26 44.45 0)
 			(effects
 				(font
@@
 		(pin "2"
 		)
+		(pin "3"
+		)
+		(pin "6"
+		)
 		(pin "5"
+		)
+		(pin "1"
 		)
 		(pin "4"
 		)
-		(pin "6"
-		)
-		(pin "1"
-		)
-		(pin "3"
-		)
 		(instances
-			(project "power_distribution"
+			(project ""
 				(path "/60722063-abcd-445d-bfe3-2bc3b4deef0d/b718a78d-1366-440c-a3b7-c9fe281beaec"
-					(reference "U?")
+					(reference "U1")
 					(unit 1)
 				)
