File: power_distribution/hw/power_distribution/stage2.kicad_sch (KiCad schematic)
At the start: 1 part

Commit message: Finish output stage
Parts:
- gave numbers to parts that had none: 1
Changed lines of the file:
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@@
 		(dnp no)
 		(fields_autoplaced yes)
-		(property "Reference" "U?"
+		(property "Reference" "U2"
 			(at 69.85 44.45 0)
 			(effects
@@
 			(project "power_distribution"
 				(path "/60722063-abcd-445d-bfe3-2bc3b4deef0d/e07a9241-783b-4e5c-9524-3952a51d89e7"
-					(reference "U?")
+					(reference "U2")
 					(unit 1)
 				)
