File: lights-backups/merged_lights.kicad_pcb (KiCad board)
At the start: 2 copper layers, 20 parts, among them J1 AVR-ISP-6, J3 Conn_01x02, J4 Conn_01x02, Q1 AO3400A, Q2 IRLML2803, Q3 IRLML2803, Q4 IRLML2803, Q5 IRLML2803, Q6 AO3400A, Q7 AO3400A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

Commit message: made updates with footprints and structure of schematic
Parts:
- added C1: 10uF, Capacitor_SMD:C_0805_2012Metric_Pad1.18x1.45mm_HandSolder, F.Cu at (173.4, 76.9)
- added C3: 10uF, Capacitor_SMD:C_0805_2012Metric_Pad1.18x1.45mm_HandSolder, F.Cu at (173.4, 79.9)
- added C4: 100u, Capacitor_SMD:C_0805_2012Metric_Pad1.18x1.45mm_HandSolder, F.Cu at (173.4, 82.9)
- added C5: 10u, Capacitor_SMD:C_0805_2012Metric_Pad1.18x1.45mm_HandSolder, F.Cu at (173.4, 85.9)
- added D1: ~, MP-3030-12ZH-30-80:LED_MP-3030-12ZH-30-80, F.Cu at (212.8, 85.2)
- added D1: RED, AB-EZD10C-A3-K65:ABEZD10CA3K65, F.Cu at (213.4, 52.4)
- added D10: RED, AB-EZD03-RA3:ABEZD03RA3, F.Cu at (213.4, 79.7)
- added D10: ~, MP-3030-12ZH-30-80:LED_MP-3030-12ZH-30-80, F.Cu at (212.8, 107.9)
- added D11: ~, MP-3030-12ZH-30-80:LED_MP-3030-12ZH-30-80, F.Cu at (195.4, 105.9)
- added D2: RED, AB-EZD10C-A3-K65:ABEZD10CA3K65, F.Cu at (195.4, 101.3)
- added D3: RED, MP-3030-12ZH-30-80:LED_MP-3030-12ZH-30-80, F.Cu at (212.8, 89.7)
- added D3: RED, AB-EZD10C-A3-K65:ABEZD10CA3K65, F.Cu at (213.4, 57.0)
- added D4: RED, AB-EZD10C-A3-K65:ABEZD10CA3K65, F.Cu at (213.4, 61.5)
- added D4: RED, MP-3030-12ZH-30-80:LED_MP-3030-12ZH-30-80, F.Cu at (212.8, 94.2)
- added D5: RED, MP-3030-12ZH-30-80:LED_MP-3030-12ZH-30-80, F.Cu at (212.8, 98.8)
- added D5: RED, AB-EZD03-RA3:ABEZD03RA3, F.Cu at (213.4, 66.0)
- added D7: RED, AB-EZD03-RA3:ABEZD03RA3, F.Cu at (213.4, 70.6)
- added D9: ~, MP-3030-12ZH-30-80:LED_MP-3030-12ZH-30-80, F.Cu at (212.8, 103.3)
- added D9: RED, AB-EZD03-RA3:ABEZD03RA3, F.Cu at (213.4, 75.2)
- added J10: Conn_01x02, Connector_JST:JST_PH_B2B-PH-K_1x02_P2.00mm_Vertical, F.Cu at (230.9, 87.7)
- added J11: Conn_01x02, Connector_JST:JST_PH_B2B-PH-K_1x02_P2.00mm_Vertical, F.Cu at (238.9, 68.0)
- added J12: Conn_01x02, Connector_JST:JST_PH_B2B-PH-K_1x02_P2.00mm_Vertical, F.Cu at (238.9, 74.6)
- added J13: Conn_01x02, Connector_JST:JST_PH_B2B-PH-K_1x02_P2.00mm_Vertical, F.Cu at (238.9, 81.2)
- added J14: Conn_01x02, Connector_JST:JST_PH_B2B-PH-K_1x02_P2.00mm_Vertical, F.Cu at (238.9, 87.7)
- added J15: Conn_01x02, Connector_JST:JST_PH_B2B-PH-K_1x02_P2.00mm_Vertical, F.Cu at (246.8, 68.0)
- added J16: Conn_01x02, Connector_JST:JST_PH_B2B-PH-K_1x02_P2.00mm_Vertical, F.Cu at (246.8, 74.6)
- added J17: Conn_01x02, Connector_JST:JST_PH_B2B-PH-K_1x02_P2.00mm_Vertical, F.Cu at (246.8, 81.2)
- added J18: Conn_01x02, Connector_JST:JST_PH_B2B-PH-K_1x02_P2.00mm_Vertical, F.Cu at (246.8, 87.7)
- added J19: Conn_01x02, Connector_JST:JST_PH_B2B-PH-K_1x02_P2.00mm_Vertical, F.Cu at (254.8, 68.0)
- added J2: Conn_01x02, Connector_JST:JST_PH_B2B-PH-K_1x02_P2.00mm_Vertical, F.Cu at (178.8, 78.1)
- added J20: Conn_01x02, Connector_JST:JST_PH_B2B-PH-K_1x02_P2.00mm_Vertical, F.Cu at (254.8, 74.6)
- added J21: Conn_01x02, Connector_JST:JST_PH_B2B-PH-K_1x02_P2.00mm_Vertical, F.Cu at (254.8, 81.2)
- added J22: Conn_01x02, Connector_JST:JST_PH_B2B-PH-K_1x02_P2.00mm_Vertical, F.Cu at (254.8, 87.7)
- added J5: Conn_01x02, Connector_JST:JST_PH_B2B-PH-K_1x02_P2.00mm_Vertical, F.Cu at (187.6, 84.2)
- added J6: Conn_01x02, Connector_JST:JST_PH_B2B-PH-K_1x02_P2.00mm_Vertical, F.Cu at (187.6, 90.8)
- added J7: Conn_01x02, Connector_JST:JST_PH_B2B-PH-K_1x02_P2.00mm_Vertical, F.Cu at (230.9, 68.0)
- added J8: Conn_01x02, Connector_JST:JST_PH_B2B-PH-K_1x02_P2.00mm_Vertical, F.Cu at (230.9, 74.6)
- added J9: Conn_01x02, Connector_JST:JST_PH_B2B-PH-K_1x02_P2.00mm_Vertical, F.Cu at (230.9, 81.2)
- added Q1: AO3400A, Package_TO_SOT_SMD:SOT-23, F.Cu at (217.4, 52.4)
- added Q2: AO3400A, Package_TO_SOT_SMD:SOT-23, F.Cu at (217.4, 56.8)
- added Q3: AO3400A, Package_TO_SOT_SMD:SOT-23, F.Cu at (222.3, 52.4)
- added Q4: AO3400A, Package_TO_SOT_SMD:SOT-23, F.Cu at (222.3, 56.8)
- added Q5: AO3400A, Package_TO_SOT_SMD:SOT-23, F.Cu at (227.3, 52.4)
- added Q6: AO3400A, Package_TO_SOT_SMD:SOT-23, F.Cu at (227.3, 56.8)
- added Q7: AO3400A, Package_TO_SOT_SMD:SOT-23, F.Cu at (232.2, 52.4)
- added Q8: AO3400A, Package_TO_SOT_SMD:SOT-23, F.Cu at (232.2, 56.8)
- added R13: 100, Resistor_SMD:R_0805_2012Metric_Pad1.20x1.40mm_HandSolder, F.Cu at (178.2, 83.4)
Connections:
- net /Headlight_1 renamed /HLED1
- net /Headlight_3 renamed /HLED3
- net /Headlight_4 renamed /HLED4
- net /LED1 renamed /TLED1
- net /LED2 renamed /TLED2
- net /LED3 renamed /TLED3
- net /LED4 renamed /TLED4
- U1 pad 11: /button2 -> /Button1
- U1 pad 12: /button1 -> unconnected-(U1-PB0-Pad12)
- U1 pad 13: unconnected-(U1-PB1-Pad13) -> /Button2
- U1 pad 24: /Headlight_2 -> /HLED2
