File: telemetry/hw/telemetry/TelemetryPCB.kicad_sch (KiCad schematic)
At the start: 12 parts, among them J1 Conn_01x06_Pin, J2 Conn_01x02_Socket, J3 Conn_01x03, J4 Conn_01x03, SW1 SW_Push, SW2 SW_Push, U1 ESP32-WROOM-32

Commit message: improved
Parts:
- removed J2: Conn_01x02_Socket, symbol Connector:Conn_01x02_Socket
- added C4: 0.1uF, symbol Device:C_Small
Connections:
- net BOOT: now also C4.1
- net GND: now also C4.2
Other:
- note removed: "Power"
- moved on the sheet: C1, J1, J3, J4, R1, R2, SW1, SW2
